Commit message: revised p3at.urdf.xacro

File: p3at_description/urdf/p3at.urdf.xacro (robot description, xacro)
@@ -13,5 +13,5 @@
   <!--rplidar link-->
   <xacro:rplidar_a2 parent="base_link" >
-    <origin xyz="0.2 0.0 0.274" rpy="0 0 ${PI}" />
+    <origin xyz="0.217 0.0 0.274" rpy="0 0 ${PI}" />
   </xacro:rplidar_a2>
 </robot>
